File: hardware/snapfob-4.sch (KiCad schematic (older format))
At the start: 6 parts, among them SW1 SW_PUSH, SW2 SW_PUSH, SW3 SW_PUSH, SW4 SW_PUSH, U1 SM200

Commit message: Pull CLKI low per datasheet.
Parts:
- BT1: footprint (none) -> _CrumpPrints:CR2032_HOLDER
- SW1, SW2, SW3, SW4: footprint (none) -> _CrumpPrints:6x6mm_pushbutton_smd
- U1: footprint (none) -> _CrumpPrints:SM200
Connections:
- net GND: now also U1.G1 (CLKI)
Changed lines of the file:
@@
 F 0 "SW1" H 6650 2460 50  0000 C CNN
 F 1 "SW_PUSH" H 6500 2270 50  0000 C CNN
-F 2 "" H 6500 2350 60  0000 C CNN
+F 2 "_CrumpPrints:6x6mm_pushbutton_smd" H 6500 2350 60  0001 C CNN
 F 3 "" H 6500 2350 60  0000 C CNN
 	1    6500 2350
@@
 F 0 "U1" H 4650 4800 60  0000 C CNN
 F 1 "SM200" H 4650 950 60  0000 C CNN
-F 2 "" H 5350 4350 60  0000 C CNN
+F 2 "_CrumpPrints:SM200" H 5350 4350 60  0001 C CNN
 F 3 "" H 5350 4350 60  0000 C CNN
 	1    4650 3100
@@
 F 0 "SW2" H 6650 2860 50  0000 C CNN
 F 1 "SW_PUSH" H 6500 2670 50  0000 C CNN
-F 2 "" H 6500 2750 60  0000 C CNN
+F 2 "_CrumpPrints:6x6mm_pushbutton_smd" H 6500 2750 60  0001 C CNN
 F 3 "" H 6500 2750 60  0000 C CNN
 	1    6500 2750
@@
 F 0 "SW3" H 6650 3260 50  0000 C CNN
 F 1 "SW_PUSH" H 6500 3070 50  0000 C CNN
-F 2 "" H 6500 3150 60  0000 C CNN
+F 2 "_CrumpPrints:6x6mm_pushbutton_smd" H 6500 3150 60  0001 C CNN
 F 3 "" H 6500 3150 60  0000 C CNN
 	1    6500 3150
@@
 F 0 "SW4" H 6650 3660 50  0000 C CNN
 F 1 "SW_PUSH" H 6500 3470 50  0000 C CNN
-F 2 "" H 6500 3550 60  0000 C CNN
+F 2 "_CrumpPrints:6x6mm_pushbutton_smd" H 6500 3550 60  0001 C CNN
 F 3 "" H 6500 3550 60  0000 C CNN
 	1    6500 3550
@@
 F 0 "BT1" H 2600 2050 50  0000 C CNN
 F 1 "BATTERY" H 2600 1660 50  0000 C CNN
-F 2 "" H 2600 1850 60  0000 C CNN
+F 2 "_CrumpPrints:CR2032_HOLDER" H 2600 1850 60  0001 C CNN
 F 3 "" H 2600 1850 60  0000 C CNN
 	1    2600 1850
@@
 Connection ~ 3700 2650
 $Comp
-L PWR_FLAG #FLG?
+L PWR_FLAG #FLG06
 U 1 1 56C0F343
 P 2250 1900
-F 0 "#FLG?" H 2250 1995 30  0001 C CNN
+F 0 "#FLG06" H 2250 1995 30  0001 C CNN
 F 1 "PWR_FLAG" H 2250 2080 30  0000 C CNN
 F 2 "" H 2250 1900 60  0000 C CNN
@@
 $EndComp
 $Comp
-L PWR_FLAG #FLG?
+L PWR_FLAG #FLG07
 U 1 1 56C0F375
 P 2950 1800
-F 0 "#FLG?" H 2950 1895 30  0001 C CNN
+F 0 "#FLG07" H 2950 1895 30  0001 C CNN
 F 1 "PWR_FLAG" H 2950 1980 30  0000 C CNN
 F 2 "" H 2950 1800 60  0000 C CNN
@@
 	2250 1900 2250 1850
 Connection ~ 2250 1850
+$Comp
+L GND #PWR?
+U 1 1 56C165A4
+P 3800 3150
+F 0 "#PWR?" H 3800 3150 30  0001 C CNN
+F 1 "GND" H 3800 3080 30  0001 C CNN
+F 2 "" H 3800 3150 60  0000 C CNN
+F 3 "" H 3800 3150 60  0000 C CNN
+	1    3800 3150
+	1    0    0    -1
+$EndComp
+Wire Wire Line
+	3800 3150 3800 3050
+Wire Wire Line
+	3800 3050 3900 3050
 $EndSCHEMATC
